File: gconsole.kicad_sch (KiCad schematic)
At the start: 3 parts, among them SW1 SW_Push, U1 XIAO-ESP32-C3-DIP

Commit message: Finished designing PCB
Parts:
- removed U1: XIAO-ESP32-C3-DIP, Seeed Studio XIAO Series Library:XIAO-ESP32C3-DIP, symbol Seeed_Studio_XIAO_Series:XIAO-ESP32-C3-DIP
- added H1, H2, H3, H4: MountingHole, MountingHole:MountingHole_3.2mm_M3, symbol Mechanical:MountingHole
- added J1: Conn_01x07_Socket, Connector_PinHeader_2.54mm:PinHeader_1x07_P2.54mm_Vertical, symbol Connector:Conn_01x07_Socket
- added S1: EG1271A, EG1271, symbol EG1271A:EG1271A
- added TP1, TP2: TestPoint, TestPoint:TestPoint_Pad_D4.0mm, symbol Connector:TestPoint
- added U1: XIAO-ESP32-C3-SMD, Seeed Studio XIAO Series Library:XIAO-ESP32C3-SMD-modified, symbol Seeed_Studio_XIAO_Series:XIAO-ESP32-C3-SMD
Connections:
- net at SW1.1: now also U1.8 (GPIO20_D7_RX)
- net GND: now reaches SW1.2
- net GND: now also VR1.A1 (CCW_1), VR1.B1 (CCW_2), J1.7 (Pin_7), TP1.1, U1.13 (GND), U1.16 (GND), U1.20 (GND)
- net at VR1.A2 (WIPER_1): now also U1.1 (GPIO2_A0_D0)
- net +3V3: now reaches VR1.A3 (CW_1)
- net +3V3: now also VR1.B3 (CW_2), J1.6 (Pin_6), U1.12 (3V3)
- net at VR1.B2 (WIPER_2): now also U1.2 (GPIO3_A1_D1)
- new net: S1.3 (NO_1), U1.15 (BAT)
- new net: J1.1 (Pin_1), U1.7 (GPIO21_D6_TX)
- new net: J1.2 (Pin_2), U1.6 (GPIO7_D5_SCL)
- new net: J1.3 (Pin_3), U1.5 (GPIO6_D4_SDA)
- new net: J1.4 (Pin_4), U1.11 (GPIO10_D10_MOSI)
- new net: J1.5 (Pin_5), U1.9 (GPIO8_D8_SCK)
- new net +BAT: S1.2 (COM_1), TP2.1
Other:
- moved on the sheet: SW1, VR1
